File: Amber.sch (KiCad schematic (older format))
At the start: 73 parts, among them CN480 DB15-VGA, J481 Conn_01x03, J482 Conn_01x03, J483 Conn_01x03, SW481 SW_DIP_x01, U470 MSM514221RS-6, U471 MSM514221RS-6, U472 MSM514221RS-6, U473 uPD42101C-2, U474 uPD42101C-2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

Commit message: Updated footprint library
Parts:
- C483: footprint Capacitor_Tantalum_SMD:CP_EIA-3216-18_Kemet-A_Pad1.58x1.35mm_HandSolder -> A3000:CP_EIA-3528-12_Kemet-T_Pad1.50x2.35mm_HandSolder
Changed lines of the file:
@@
 F 0 "C483" V 5350 10000 50  0000 C CNN
 F 1 "10uF(Tan)" V 5650 10050 50  0000 C CNN
-F 2 "Capacitor_Tantalum_SMD:CP_EIA-3216-18_Kemet-A_Pad1.58x1.35mm_HandSolder" H 5538 9900 50  0001 C CNN
+F 2 "A3000:CP_EIA-3528-12_Kemet-T_Pad1.50x2.35mm_HandSolder" H 5538 9900 50  0001 C CNN
 F 3 "~" H 5500 10050 50  0001 C CNN
 	1    5500 10050
